File: KiCad/pulsegen_outdoor/pulsegen_outdoor.sch (KiCad schematic (older format))
At the start: 31 parts, among them J1 Conn_Coaxial, J2 Conn_Coaxial, Q1 MMBT3904, U1 ADCMP572, U2 LT1963AxST-3.3

Commit message: Update schematics
Parts:
- removed C7: 68p, Capacitors_SMD:C_1206_HandSoldering, symbol Device:C
- removed C8: 10p, Capacitors_SMD:C_1206_HandSoldering, symbol Device:C
- removed D2: SMS7630-079LF, Diodes_SMD:D_SC-80_HandSoldering, symbol Device:D
- removed Q1: MMBT3904, TO_SOT_Packages_SMD:SOT-23_Handsoldering, symbol Transistor_BJT:MMBT3904
- removed R6: 310, Resistors_SMD:R_1206_HandSoldering, symbol Device:R
- removed R7: 560, Resistors_SMD:R_1206_HandSoldering, symbol Device:R
- removed R8: 510, Resistors_SMD:R_1206_HandSoldering, symbol Device:R
- removed R9: 10k, Resistors_SMD:R_1206_HandSoldering, symbol Device:R
- added C11: 1u, Capacitor_SMD:C_1206_3216Metric_Pad1.42x1.75mm_HandSolder, symbol Device:C
- added C4: 10n, Capacitor_SMD:C_1206_3216Metric_Pad1.42x1.75mm_HandSolder, symbol Device:C
- added H1, H2, H3, H4: MountingHole, MountingHole:MountingHole_3.2mm_M3_DIN965, symbol Mechanical:MountingHole
- added TP2: VP, TestPoint:TestPoint_THTPad_D1.0mm_Drill0.5mm, symbol Connector:TestPoint
- added TP3: VN, TestPoint:TestPoint_THTPad_D1.0mm_Drill0.5mm, symbol Connector:TestPoint
- C1, C2, C3: footprint Capacitors_SMD:C_1206_HandSoldering -> Capacitor_SMD:C_1206_3216Metric_Pad1.42x1.75mm_HandSolder
- C10: renamed from C11; footprint Capacitors_SMD:C_1206_HandSoldering -> Capacitor_SMD:C_1206_3216Metric_Pad1.42x1.75mm_HandSolder
- C5: renamed from C4; footprint Capacitors_SMD:C_1206_HandSoldering -> Capacitor_SMD:C_1206_3216Metric_Pad1.42x1.75mm_HandSolder
- C6: renamed from C5; value CP -> 10u; footprint Capacitors_Tantalum_SMD:CP_Tantalum_Case-B_EIA-3528-21_Hand -> Capacitor_Tantalum_SMD:CP_EIA-3528-21_Kemet-B_Pad1.50x2.35mm_HandSolder
- C7: renamed from C6; value CP -> 10u; footprint Capacitors_Tantalum_SMD:CP_Tantalum_Case-B_EIA-3528-21_Hand -> Capacitor_Tantalum_SMD:CP_EIA-3528-21_Kemet-B_Pad1.50x2.35mm_HandSolder
- C8: renamed from C9; footprint Capacitors_SMD:C_1206_HandSoldering -> Capacitor_SMD:C_1206_3216Metric_Pad1.42x1.75mm_HandSolder
- C9: renamed from C10; footprint Capacitors_SMD:C_1206_HandSoldering -> Capacitor_SMD:C_1206_3216Metric_Pad1.42x1.75mm_HandSolder
- D1: footprint TO_SOT_Packages_SMD:SOT-23 -> Package_TO_SOT_SMD:SOT-23
- J1, J2: footprint Connectors:SMA_THT_Jack_Straight -> Connector_Coaxial:SMA_Molex_73251-1153_EdgeMount_Horizontal
- L1: value 10u -> 100u; footprint Inductors_SMD:L_1210_HandSoldering -> Inductor_SMD:L_1210_3225Metric_Pad1.42x2.65mm_HandSolder
- R1, R2, R3, R4, R5: footprint Resistors_SMD:R_1206_HandSoldering -> Resistor_SMD:R_1206_3216Metric_Pad1.42x1.75mm_HandSolder
- TP1: footprint (none) -> TestPoint:TestPoint_THTPad_D1.0mm_Drill0.5mm
- TP4: renamed from TP2; footprint (none) -> TestPoint:TestPoint_THTPad_D1.0mm_Drill0.5mm
- TP5: renamed from TP3; footprint (none) -> TestPoint:TestPoint_THTPad_D1.0mm_Drill0.5mm
- U1: footprint Housings_CSP:LFCSP-16-1EP_3x3mm_Pitch0.5mm -> Package_CSP:LFCSP-16-1EP_3x3mm_P0.5mm_EP1.7x1.7mm_ThermalVias
Connections:
- net +3V3: now also C11.2
- net GND: now also C11.1, C4.1; no longer U1.1 (VTP)
- net at C2.1, U1.2 (VP): now also TP2.1; no longer R1.1
- net at U1.3 (VN): now also R1.1, U1.1 (VTP), C4.2, TP3.1
- no-connect marks 1 -> 2
Other:
- note added: "Datasheet: the latch function can be disabled\nby leaving LE unconnected and connecting ~LE\nto ground via 750 ohm resistor."
- note removed: "The connection to VN is unfinished business..."
- moved on the sheet: C10, C8, C9, R1
