File: KiCad/pulsegen_indoor/pulsegen_indoor.kicad_pcb (KiCad board)
At the start: 2 copper layers, 75 x 50 mm, 37 parts, among them J1 USB-serial, J2 10MHz reference, J3 12V, J4 Conn_Coaxial, J5 GND, U1 LM2940, U2 TLX9310, U3 TLX9310, U4 OPA692, U5 TPS22810

Commit message: Changes after prototyping
Parts:
- J5: value GND -> Scope ground
- R1, R2: value R -> 510
- moved R6 10.3 mm to (145.2, 114.9)
- moved D2 5.72 mm to (135.9, 117.5)
Connections:
- C1 pad 1: PulseGen12V -> +12V
- U1 pad 1: PulseGen12V -> +12V
Routing:
- net +12V: track 19.1 -> 34.4 mm
- net PulseGen12V: track 92.0 -> 77.4 mm
- net Net-(D2-Pad2): track 15.3 -> 7.82 mm
- net GND: track 65.5 -> 71.3 mm
Other:
- board text added: "Ozone radiometer Harmonic generator - indoor unit MS/UNIS/2021-XX-YY"
- board text added: "RTS"
- board text removed: "Ozone radiometer Harmonic generator - indoor unit MS/UNIS/2020-12-14"
